Commit message: [FMT] Remove deprecated --inorder parameter and general formatting improvements

File: urdf/_d435.gazebo.xacro (robot description, xacro)
@@ -6,5 +6,8 @@
 -->
 <robot xmlns:xacro="http://ros.org/wiki/xacro">
-  <xacro:macro name="gazebo_d435" params="camera_name reference_link topics_ns depth_optical_frame color_optical_frame infrared1_optical_frame infrared2_optical_frame publish_pointcloud:=true" >
+  <xacro:macro
+    name="gazebo_d435"
+    params="camera_name reference_link topics_ns depth_optical_frame color_optical_frame infrared1_optical_frame
+            infrared2_optical_frame publish_pointcloud:=true" >
     <!-- Load parameters to model's main link-->
     <xacro:property name="deg_to_rad" value="0.01745329251994329577" />

File: urdf/_d435.urdf.xacro (robot description, xacro)
@@ -9,5 +9,7 @@
   <!--File includes-->
   <xacro:include filename="$(find realsense2_description)/urdf/_d435.gazebo.xacro"/>
-  <xacro:macro name="sensor_d435" params="name:=camera topics_ns:=camera parent *origin publish_pointcloud:=true">
+  <xacro:macro
+    name="sensor_d435"
+    params="name:=camera topics_ns:=camera parent *origin publish_pointcloud:=true">
     <xacro:property name="M_PI" value="3.1415926535897931" />
     <!-- The following values are approximate, and the camera node
@@ -119,5 +121,9 @@
     <link name="${name}_color_optical_frame"/>
     <!-- Realsense Gazebo Plugin -->
-    <xacro:gazebo_d435 camera_name="${name}" reference_link="${name}_link" topics_ns="${topics_ns}" depth_optical_frame="${name}_depth_optical_frame" color_optical_frame="${name}_color_optical_frame" infrared1_optical_frame="${name}_left_ir_optical_frame" infrared2_optical_frame="${name}_right_ir_optical_frame" publish_pointcloud="${publish_pointcloud}"/>
+    <xacro:gazebo_d435
+        camera_name="${name}" reference_link="${name}_link" topics_ns="${topics_ns}"
+        depth_optical_frame="${name}_depth_optical_frame" color_optical_frame="${name}_color_optical_frame"
+        infrared1_optical_frame="${name}_left_ir_optical_frame" infrared2_optical_frame="${name}_right_ir_optical_frame"
+        publish_pointcloud="${publish_pointcloud}"/>
   </xacro:macro>
 </robot>

File: urdf/test_d435_camera.urdf.xacro (robot description, xacro)
@@ -3,5 +3,9 @@
   <xacro:include filename="$(find realsense2_description)/urdf/_d435.urdf.xacro" />
   <link name="base_link" />
-  <xacro:sensor_d435 name="camera" topics_ns="camera" parent="base_link" publish_pointcloud="true">
+  <xacro:sensor_d435
+      name="camera"
+      topics_ns="camera"
+      parent="base_link"
+      publish_pointcloud="true">
     <origin xyz="0 0 0" rpy="0 0 0" />
   </xacro:sensor_d435>
